File: flow/designs/h.r.3.3/kinase_kicad/component.kicad_sch (KiCad schematic)
At the start: 22 parts

Commit message: Update kinase kicad example
Parts:
- P1, P3, V10, V11, V2, V3, V4, V5, V8, V9: footprint (none) -> h.r.3.3:valve_80px_1
- P2: footprint (none) -> h.r.3.3:pump_40px_0
- R1: footprint (none) -> h.r.3.3:inline_res_40nl
- V1, V10, V11, V12, V13, V14, V15, V2, V3, V4, V5, V6, V8, V9: footprint h.r.3.3:valve_20px_1 -> h.r.3.3:valve_80px_1
- V7: footprint h.r.3.3:mux3_20px_0 -> (none)
Changed lines of the file:
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@@
 			)
 		)
-		(property "Footprint" "h.r.3.3:valve_20px_1"
+		(property "Footprint" "h.r.3.3:valve_80px_1"
 			(at 101.6 185.42 0)
 			(hide yes)
@@
 			)
 		)
-		(property "Footprint" "h.r.3.3:valve_20px_1"
+		(property "Footprint" "h.r.3.3:valve_80px_1"
 			(at 96.52 185.42 0)
 			(hide yes)
@@
 			)
 		)
-		(property "Footprint" ""
+		(property "Footprint" "h.r.3.3:valve_80px_1"
 			(at 76.2 185.42 0)
 			(hide yes)
@@
 			)
 		)
-		(property "Footprint" "h.r.3.3:valve_20px_1"
+		(property "Footprint" "h.r.3.3:valve_80px_1"
 			(at 262.89 100.33 0)
 			(hide yes)
@@
 			)
 		)
-		(property "Footprint" ""
+		(property "Footprint" "h.r.3.3:valve_80px_1"
 			(at 101.6 102.87 0)
 			(hide yes)
@@
 			)
 		)
-		(property "Footprint" ""
+		(property "Footprint" "h.r.3.3:valve_80px_1"
 			(at 166.37 60.96 0)
 			(hide yes)
@@
 			)
 		)
-		(property "Footprint" ""
+		(property "Footprint" "h.r.3.3:pump_40px_0"
 			(at 137.16 110.49 0)
 			(hide yes)
@@
 			)
 		)
-		(property "Footprint" ""
+		(property "Footprint" "h.r.3.3:valve_80px_1"
 			(at 114.3 60.96 0)
 			(hide yes)
@@
 			)
 		)
-		(property "Footprint" "h.r.3.3:valve_20px_1"
+		(property "Footprint" "h.r.3.3:valve_80px_1"
 			(at 71.12 185.42 0)
 			(hide yes)
@@
 			)
 		)
-		(property "Footprint" ""
+		(property "Footprint" "h.r.3.3:valve_80px_1"
 			(at 154.94 60.96 0)
 			(hide yes)
@@
 			)
 		)
-		(property "Footprint" "h.r.3.3:valve_20px_1"
+		(property "Footprint" "h.r.3.3:valve_80px_1"
 			(at 238.76 102.87 0)
 			(hide yes)
@@
 			)
 		)
-		(property "Footprint" "h.r.3.3:valve_20px_1"
+		(property "Footprint" "h.r.3.3:valve_80px_1"
 			(at 93.98 185.42 0)
 			(hide yes)
@@
 			)
 		)
-		(property "Footprint" "h.r.3.3:valve_20px_1"
+		(property "Footprint" "h.r.3.3:valve_80px_1"
 			(at 179.07 60.96 0)
 			(hide yes)
@@
 			)
 		)
-		(property "Footprint" "h.r.3.3:valve_20px_1"
+		(property "Footprint" "h.r.3.3:valve_80px_1"
 			(at 73.66 185.42 0)
 			(hide yes)
@@
 			)
 		)
-		(property "Footprint" "h.r.3.3:valve_20px_1"
+		(property "Footprint" "h.r.3.3:valve_80px_1"
 			(at 173.99 90.17 0)
 			(hide yes)
@@
 			)
 		)
-		(property "Footprint" ""
+		(property "Footprint" "h.r.3.3:inline_res_40nl"
 			(at 146.304 68.326 0)
 			(hide yes)
@@
 			)
 		)
-		(property "Footprint" "h.r.3.3:valve_20px_1"
+		(property "Footprint" "h.r.3.3:valve_80px_1"
 			(at 204.47 102.87 0)
 			(hide yes)
@@
 			)
 		)
-		(property "Footprint" ""
+		(property "Footprint" "h.r.3.3:valve_80px_1"
 			(at 127 60.96 0)
 			(hide yes)
@@
 			)
 		)
-		(property "Footprint" "h.r.3.3:valve_20px_1"
+		(property "Footprint" "h.r.3.3:valve_80px_1"
 			(at 256.54 111.76 0)
 			(hide yes)
@@
 			)
 		)
-		(property "Footprint" "h.r.3.3:valve_20px_1"
+		(property "Footprint" "h.r.3.3:valve_80px_1"
 			(at 81.28 185.42 0)
 			(hide yes)
@@
 			)
 		)
-		(property "Footprint" "h.r.3.3:valve_20px_1"
+		(property "Footprint" "h.r.3.3:valve_80px_1"
 			(at 93.98 60.96 0)
 			(hide yes)
@@
 			)
 		)
-		(property "Footprint" ""
+		(property "Footprint" "h.r.3.3:valve_80px_1"
 			(at 78.74 185.42 0)
 			(hide yes)
@@
 			)
 		)
-		(property "Footprint" "h.r.3.3:mux3_20px_0"
+		(property "Footprint" ""
 			(at 87.63 60.96 0)
 			(hide yes)
@@
 			)
 		)
-		(property "Footprint" "h.r.3.3:valve_20px_1"
+		(property "Footprint" "h.r.3.3:valve_80px_1"
 			(at 194.31 102.87 0)
 			(hide yes)
@@
 			)
 		)
-		(property "Footprint" ""
+		(property "Footprint" "h.r.3.3:valve_80px_1"
 			(at 91.44 185.42 0)
 			(hide yes)
@@
 			)
 		)
-		(property "Footprint" "h.r.3.3:valve_20px_1"
+		(property "Footprint" "h.r.3.3:valve_80px_1"
 			(at 83.82 185.42 0)
 			(hide yes)
@@
 			)
 		)
-		(property "Footprint" ""
+		(property "Footprint" "h.r.3.3:valve_80px_1"
 			(at 106.68 60.96 0)
 			(hide yes)
@@
 			)
 		)
-		(property "Footprint" "h.r.3.3:valve_20px_1"
+		(property "Footprint" "h.r.3.3:valve_80px_1"
 			(at 68.58 185.42 0)
 			(hide yes)
@@
 			)
 		)
-		(property "Footprint" "h.r.3.3:valve_20px_1"
+		(property "Footprint" "h.r.3.3:valve_80px_1"
 			(at 99.06 185.42 0)
 			(hide yes)
@@
 			)
 		)
-		(property "Footprint" "h.r.3.3:valve_20px_1"
+		(property "Footprint" "h.r.3.3:valve_80px_1"
 			(at 179.07 110.49 0)
 			(hide yes)
@@
 			)
 		)
-		(property "Footprint" ""
+		(property "Footprint" "h.r.3.3:valve_80px_1"
 			(at 88.9 185.42 0)
 			(hide yes)
@@
 			)
 		)
-		(property "Footprint" "h.r.3.3:valve_20px_1"
+		(property "Footprint" "h.r.3.3:valve_80px_1"
 			(at 86.36 185.42 0)
 			(hide yes)
@@
 			)
 		)
-		(property "Footprint" "h.r.3.3:valve_20px_1"
+		(property "Footprint" "h.r.3.3:valve_80px_1"
 			(at 191.77 60.96 0)
 			(hide yes)
