File: flow/designs/h.r.3.3/kinase_kicad/kinase_kicad.kicad_sch (KiCad schematic)
At the start: 32 parts

Commit message: Update kinase kicad example
Parts:
- J1, J2, J27, J28, J29, J3, J30, J31, J4: footprint h.r.3.3:pinhole_325px_met5 -> h.r.3.3:pinhole_325px_0
- J10, J11, J12, J13, J14, J15, J16, J17, J18, J19, J20, J21, J22, J23, J24, J25, J26, J5, J6, J7, J8, J9: footprint (none) -> h.r.3.3:flush_hole_0
- J32: footprint h.r.3.3:interconnect_4x8 -> h.r.3.3:interconnect_8x4
Changed lines of the file:
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@@
 	)
 	(bus_entry
-		(at 184.15 52.07)
+		(at 184.15 48.26)
 		(size 2.54 2.54)
 		(stroke
@@
 	(bus
 		(pts
-			(xy 184.15 30.48) (xy 184.15 52.07)
+			(xy 184.15 30.48) (xy 184.15 48.26)
 		)
 		(stroke
@@
 	(bus
 		(pts
-			(xy 246.38 20.32) (xy 246.38 64.77)
+			(xy 246.38 24.13) (xy 246.38 64.77)
 		)
 		(stroke
@@
 	(wire
 		(pts
-			(xy 186.69 54.61) (xy 231.14 54.61)
+			(xy 186.69 50.8) (xy 231.14 50.8)
 		)
 		(stroke
@@
 	(wire
 		(pts
-			(xy 231.14 54.61) (xy 231.14 59.69)
+			(xy 231.14 50.8) (xy 231.14 59.69)
 		)
 		(stroke
@@
 	(bus
 		(pts
-			(xy 105.41 20.32) (xy 105.41 48.26)
+			(xy 105.41 24.13) (xy 105.41 48.26)
 		)
 		(stroke
@@
 	(bus
 		(pts
-			(xy 184.15 52.07) (xy 184.15 57.15)
+			(xy 184.15 48.26) (xy 184.15 57.15)
 		)
 		(stroke
@@
 	(bus
 		(pts
-			(xy 246.38 20.32) (xy 105.41 20.32)
+			(xy 246.38 24.13) (xy 105.41 24.13)
 		)
 		(stroke
@@
 	)
 	(label "pump5"
-		(at 203.2 54.61 0)
+		(at 194.31 50.8 0)
 		(effects
 			(font
@@
 			)
 		)
-		(property "Footprint" ""
+		(property "Footprint" "h.r.3.3:flush_hole_0"
 			(at 80.01 151.13 0)
 			(hide yes)
@@
 			)
 		)
-		(property "Footprint" ""
+		(property "Footprint" "h.r.3.3:flush_hole_0"
 			(at 129.54 140.97 0)
 			(hide yes)
@@
 			)
 		)
-		(property "Footprint" ""
+		(property "Footprint" "h.r.3.3:flush_hole_0"
 			(at 129.54 143.51 0)
 			(hide yes)
@@
 			)
 		)
-		(property "Footprint" ""
+		(property "Footprint" "h.r.3.3:flush_hole_0"
 			(at 129.54 161.29 0)
 			(hide yes)
@@
 			)
 		)
-		(property "Footprint" ""
+		(property "Footprint" "h.r.3.3:flush_hole_0"
 			(at 129.54 146.05 0)
 			(hide yes)
@@
 			)
 		)
-		(property "Footprint" ""
+		(property "Footprint" "h.r.3.3:flush_hole_0"
 			(at 129.54 148.59 0)
 			(hide yes)
@@
 			)
 		)
-		(property "Footprint" "h.r.3.3:pinhole_325px_met5"
+		(property "Footprint" "h.r.3.3:pinhole_325px_0"
 			(at 59.69 46.99 0)
 			(hide yes)
@@
 			)
 		)
-		(property "Footprint" ""
+		(property "Footprint" "h.r.3.3:flush_hole_0"
 			(at 129.54 181.61 0)
 			(hide yes)
@@
 			)
 		)
-		(property "Footprint" ""
+		(property "Footprint" "h.r.3.3:flush_hole_0"
 			(at 129.54 151.13 0)
 			(hide yes)
@@
 			)
 		)
-		(property "Footprint" ""
+		(property "Footprint" "h.r.3.3:flush_hole_0"
 			(at 129.54 171.45 0)
 			(hide yes)
@@
 			)
 		)
-		(property "Footprint" "h.r.3.3:pinhole_325px_met5"
+		(property "Footprint" "h.r.3.3:pinhole_325px_0"
 			(at 161.29 105.41 0)
 			(hide yes)
@@
 			)
 		)
-		(property "Footprint" "h.r.3.3:pinhole_325px_met5"
+		(property "Footprint" "h.r.3.3:pinhole_325px_0"
 			(at 154.94 55.88 0)
 			(hide yes)
@@
 			)
 		)
-		(property "Footprint" "h.r.3.3:pinhole_325px_met5"
+		(property "Footprint" "h.r.3.3:pinhole_325px_0"
 			(at 59.69 60.96 0)
 			(hide yes)
@@
 			)
 		)
-		(property "Footprint" ""
+		(property "Footprint" "h.r.3.3:flush_hole_0"
 			(at 80.01 158.75 0)
 			(hide yes)
@@
 			)
 		)
-		(property "Footprint" ""
+		(property "Footprint" "h.r.3.3:flush_hole_0"
 			(at 129.54 163.83 0)
 			(hide yes)
@@
 			)
 		)
-		(property "Footprint" "h.r.3.3:pinhole_325px_met5"
+		(property "Footprint" "h.r.3.3:pinhole_325px_0"
 			(at 59.69 44.45 0)
 			(hide yes)
@@
 			)
 		)
-		(property "Footprint" ""
+		(property "Footprint" "h.r.3.3:flush_hole_0"
 			(at 129.54 166.37 0)
 			(hide yes)
@@
 			)
 		)
-		(property "Footprint" ""
+		(property "Footprint" "h.r.3.3:flush_hole_0"
 			(at 129.54 156.21 0)
 			(hide yes)
@@
 			)
 		)
-		(property "Footprint" ""
+		(property "Footprint" "h.r.3.3:flush_hole_0"
 			(at 80.01 153.67 0)
 			(hide yes)
@@
 			)
 		)
-		(property "Footprint" "h.r.3.3:pinhole_325px_met5"
+		(property "Footprint" "h.r.3.3:pinhole_325px_0"
 			(at 154.94 88.9 0)
 			(hide yes)
@@
 			)
 		)
-		(property "Footprint" ""
+		(property "Footprint" "h.r.3.3:flush_hole_0"
 			(at 129.54 158.75 0)
 			(hide yes)
@@
 			)
 		)
-		(property "Footprint" ""
+		(property "Footprint" "h.r.3.3:flush_hole_0"
 			(at 129.54 173.99 0)
 			(hide yes)
@@
 			)
 		)
-		(property "Footprint" ""
+		(property "Footprint" "h.r.3.3:flush_hole_0"
 			(at 129.54 168.91 0)
 			(hide yes)
@@
 			)
 		)
-		(property "Footprint" "h.r.3.3:pinhole_325px_met5"
+		(property "Footprint" "h.r.3.3:pinhole_325px_0"
 			(at 60.96 106.68 0)
 			(hide yes)
@@
 			)
 		)
-		(property "Footprint" ""
+		(property "Footprint" "h.r.3.3:flush_hole_0"
 			(at 129.54 179.07 0)
 			(hide yes)
@@
 			)
 		)
-		(property "Footprint" "h.r.3.3:pinhole_325px_met5"
+		(property "Footprint" "h.r.3.3:pinhole_325px_0"
 			(at 154.94 91.44 0)
 			(hide yes)
@@
 			)
 		)
-		(property "Footprint" ""
+		(property "Footprint" "h.r.3.3:flush_hole_0"
 			(at 80.01 148.59 0)
 			(hide yes)
@@
 			)
 		)
-		(property "Footprint" "h.r.3.3:pinhole_325px_met5"
+		(property "Footprint" "h.r.3.3:pinhole_325px_0"
 			(at 154.94 86.36 0)
 			(hide yes)
@@
 		(fields_autoplaced yes)
 		(property "Reference" "J32"
-			(at 215.5825 53.34 0)
+			(at 215.5825 54.61 0)
 			(show_name no)
 			(do_not_autoplace no)
@@
 			)
 		)
-		(property "Footprint" "h.r.3.3:interconnect_4x8"
+		(property "Footprint" "h.r.3.3:interconnect_8x4"
 			(at 222.25 97.79 0)
 			(hide yes)
@@
 			)
 		)
-		(property "Footprint" ""
+		(property "Footprint" "h.r.3.3:flush_hole_0"
 			(at 129.54 176.53 0)
 			(hide yes)
@@
 			)
 		)
-		(property "Footprint" ""
+		(property "Footprint" "h.r.3.3:flush_hole_0"
 			(at 80.01 156.21 0)
 			(hide yes)
@@
 			)
 		)
-		(property "Footprint" ""
+		(property "Footprint" "h.r.3.3:flush_hole_0"
 			(at 129.54 153.67 0)
 			(hide yes)
